File: zorionx_nivara/ANALOG_IN.kicad_sch (KiCad schematic)
At the start: 14 parts, among them Q3 IRLML0040, Q4 IRLML0040, U12 LTV-357T, U14 LTV-357T

Commit message: ultimo commit 1
Parts:
- removed D10, D29: LED ON, LED_SMD:LED_0603_1608Metric, symbol Device:LED
- removed Q3, Q4: IRLML0040, PCM_Package_TO_SOT_SMD_AKL:SOT-23, symbol PCM_Transistor_MOSFET_AKL:IRLML0040
- removed R27, R30: 100, PCM_Resistor_SMD_AKL:R_0603_1608Metric, symbol PCM_Resistor_US_AKL:R_0603
- removed R28: 30k, PCM_Resistor_SMD_AKL:R_0603_1608Metric, symbol PCM_Resistor_US_AKL:R_0603
- removed R29: 22k, PCM_Resistor_SMD_AKL:R_0603_1608Metric, symbol PCM_Resistor_US_AKL:R_0603
- removed R31: 30K, PCM_Resistor_SMD_AKL:R_0603_1608Metric, symbol PCM_Resistor_US_AKL:R_0603
- removed R32: 22K, PCM_Resistor_SMD_AKL:R_0603_1608Metric, symbol PCM_Resistor_US_AKL:R_0603
- removed R33, R56: 1.7K, PCM_Resistor_SMD_AKL:R_0603_1608Metric, symbol PCM_Resistor_US_AKL:R_0603
- removed U12, U14: LTV-357T, Package_SO:SO-4_4.4x3.6mm_P2.54mm, symbol Isolator:LTV-357T
- added C10, C12, C9: 100nF, PCM_Capacitor_SMD_AKL:C_0603_1608Metric, symbol PCM_Capacitor_US_AKL:C_0603
- added D11, D12, D13, D14, D15, D19: SMAJ5.0A, PCM_Diode_SMD_AKL:D_SMA, symbol PCM_Diode_TVS_AKL:SMAJ5.0A
- added R36: 100K, PCM_Resistor_SMD_AKL:R_0603_1608Metric, symbol PCM_Resistor_US_AKL:R_0603
- added R37, R39: 10K, PCM_Resistor_SMD_AKL:R_0603_1608Metric, symbol PCM_Resistor_US_AKL:R_0603
- added R38: 25K, PCM_Resistor_SMD_AKL:R_0603_1608Metric, symbol PCM_Resistor_US_AKL:R_0603
- added R42: 1k, PCM_Resistor_SMD_AKL:R_0603_1608Metric, symbol PCM_Resistor_US_AKL:R_0603
- added R43: 145, PCM_Resistor_SMD_AKL:R_0805_2012Metric, symbol PCM_Resistor_US_AKL:R_0805
Connections:
- new net +3.3V: D12.1 (K), D14.1 (K), D19.1 (K)
- new net A0_10_IN_1: R38.2
- new net A0_32_IN_1: R36.2
- new net A4_20_IN_1: R42.1, R43.1
- new net ESP32-S3_4-20_IN: C12.1, D11.1 (K), D19.2 (A), R42.2
- new net ESP32-S3_A0_10_IN_1: C10.1, D14.2 (A), D15.1 (K), R38.1, R39.2
- new net ESP32-S3_A0_32_IN_1: C9.1, D12.2 (A), D13.1 (K), R36.1, R37.2
- new net GND: C10.2, C12.2, C9.2, D11.2 (A), D13.2 (A), D15.2 (A), R37.1, R39.1, R43.2
Other:
- note added: "Entrada 0-10V"
- note added: "Entrada 0-32V"
- note added: "Entrada 4-20mA"
- note removed: "Salida PNP #1"
- note removed: "Salida PNP #2"

Commit message: Salvado
Changed lines of the file:
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@@
 		(dnp no)
 		(property "Reference" "D12"
-			(at 150.368 46.482 90)
+			(at 151.638 43.18 90)
 			(effects
 				(font
@@
 		)
 		(property "Value" "SMAJ5.0A"
-			(at 150.622 49.276 90)
+			(at 151.892 45.974 90)
 			(effects
 				(font

Commit message: Enrutando
Changed lines of the file:
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@@
-		)
-	)
-	(hierarchical_label "+3.3V"
-		(shape input)
-		(at 85.09 38.1 0)
-		(effects
-			(font
-				(size 1.27 1.27)
-			)
-			(justify left)
 		)
 	)
@@
 		)
 	)
-	(hierarchical_label "+3.3V"
-		(shape input)
-		(at 232.41 41.91 0)
-		(effects
-			(font
-				(size 1.27 1.27)
-			)
-			(justify left)
-		)
-	)
-	(hierarchical_label "+3.3V"
-		(shape input)
-		(at 157.48 41.91 0)
-		(effects
-			(font
-				(size 1.27 1.27)
-			)
-			(justify left)
-		)
-	)
 	(symbol
 		(lib_id "power:GND")
@@
 	)
 	(symbol
+		(lib_id "PCM_4ms_Power-symbol:+3.3V")
+		(at 157.48 41.91 270)
+		(unit 1)
+		(exclude_from_sim no)
+		(in_bom yes)
+		(on_board yes)
+		(dnp no)
+		(fields_autoplaced yes)
+		(property "Reference" "#PWR012"
+			(at 153.67 41.91 0)
+			(effects
+				(font
+					(size 1.27 1.27)
+				)
+				(hide yes)
+			)
+		)
+		(property "Value" "+3.3V"
+			(at 161.29 41.9099 90)
+			(effects
+				(font
+					(size 1.27 1.27)
+				)
+				(justify left)
+			)
+		)
+		(property "Footprint" ""
+			(at 157.48 41.91 0)
+			(effects
+				(font
+					(size 1.27 1.27)
+				)
+				(hide yes)
+			)
+		)
+		(property "Datasheet" ""
+			(at 157.48 41.91 0)
+			(effects
+				(font
+					(size 1.27 1.27)
+				)
+				(hide yes)
+			)
+		)
+		(property "Description" ""
+			(at 157.48 41.91 0)
+			(effects
+				(font
+					(size 1.27 1.27)
+				)
+				(hide yes)
+			)
+		)
+		(pin "1"
+		)
+		(instances
+			(project "zorionx_nivara"
+				(path "/c1255741-5652-463a-8cfd-bd2388ad7ef1/ee2c52cb-3406-40a8-8a05-a93f573fe34b/2fc75700-43b6-4a7e-8ac9-f536ae32b879"
+					(reference "#PWR012")
+					(unit 1)
+				)
+			)
+		)
+	)
+	(symbol
 		(lib_id "PCM_Resistor_US_AKL:R_0603")
 		(at 210.82 48.26 180)
@@
 	)
 	(symbol
+		(lib_id "PCM_4ms_Power-symbol:+3.3V")
+		(at 232.41 41.91 270)
+		(unit 1)
+		(exclude_from_sim no)
+		(in_bom yes)
+		(on_board yes)
+		(dnp no)
+		(fields_autoplaced yes)
+		(property "Reference" "#PWR025"
+			(at 228.6 41.91 0)
+			(effects
+				(font
+					(size 1.27 1.27)
+				)
+				(hide yes)
+			)
+		)
+		(property "Value" "+3.3V"
+			(at 236.22 41.9099 90)
+			(effects
+				(font
+					(size 1.27 1.27)
+				)
+				(justify left)
+			)
+		)
+		(property "Footprint" ""
+			(at 232.41 41.91 0)
+			(effects
+				(font
+					(size 1.27 1.27)
+				)
+				(hide yes)
+			)
+		)
+		(property "Datasheet" ""
+			(at 232.41 41.91 0)
+			(effects
+				(font
+					(size 1.27 1.27)
+				)
+				(hide yes)
+			)
+		)
+		(property "Description" ""
+			(at 232.41 41.91 0)
+			(effects
+				(font
+					(size 1.27 1.27)
+				)
+				(hide yes)
+			)
+		)
+		(pin "1"
+		)
+		(instances
+			(project "zorionx_nivara"
+				(path "/c1255741-5652-463a-8cfd-bd2388ad7ef1/ee2c52cb-3406-40a8-8a05-a93f573fe34b/2fc75700-43b6-4a7e-8ac9-f536ae32b879"
+					(reference "#PWR025")
+					(unit 1)
+				)
+			)
+		)
+	)
+	(symbol
 		(lib_id "PCM_Diode_TVS_AKL:SMAJ5.0A")
 		(at 80.01 58.42 270)
@@
 					(unit 1)
 				)
+			)
+		)
+	)
+	(symbol
+		(lib_id "PCM_4ms_Power-symbol:+3.3V")
+		(at 85.09 38.1 270)
+		(unit 1)
+		(exclude_from_sim no)
+		(in_bom yes)
+		(on_board yes)
+		(dnp no)
+		(fields_autoplaced yes)
+		(property "Reference" "#PWR08"
+			(at 81.28 38.1 0)
+			(effects
+				(font
+					(size 1.27 1.27)
+				)
+				(hide yes)
+			)
+		)
+		(property "Value" "+3.3V"
+			(at 88.9 38.0999 90)
+			(effects
+				(font
+					(size 1.27 1.27)
+				)
+				(justify left)
+			)
+		)
+		(property "Footprint" ""
+			(at 85.09 38.1 0)
+			(effects
+				(font
+					(size 1.27 1.27)
+				)
+				(hide yes)
+			)
+		)
+		(property "Datasheet" ""
+			(at 85.09 38.1 0)
+			(effects
+				(font
+					(size 1.27 1.27)
+				)
+				(hide yes)
+			)
+		)
+		(property "Description" ""
+			(at 85.09 38.1 0)
+			(effects
+				(font
+					(size 1.27 1.27)
+				)
+				(hide yes)
+			)
+		)
+		(pin "1"
+		)
+		(instances
+			(project ""
+				(path "/c1255741-5652-463a-8cfd-bd2388ad7ef1/ee2c52cb-3406-40a8-8a05-a93f573fe34b/2fc75700-43b6-4a7e-8ac9-f536ae32b879"
+					(reference "#PWR08")
+					(unit 1)
+				)
