File: zorionx_nivara/DIGITAL_IN.kicad_sch (KiCad schematic)
At the start: 8 parts, among them U5 LTV-357T, U6 LTV-357T

Commit message: ultimo commit 1
Parts:
- removed D2, D3: LED ON, LED_SMD:LED_0603_1608Metric, symbol Device:LED
- removed R10, R11: 1k, PCM_Resistor_SMD_AKL:R_0603_1608Metric, symbol PCM_Resistor_US_AKL:R_0603
- removed R7, R9: 180, PCM_Resistor_SMD_AKL:R_0603_1608Metric, symbol PCM_Resistor_US_AKL:R_0603
- removed U5, U6: LTV-357T, Package_SO:SO-4_4.4x3.6mm_P2.54mm, symbol Isolator:LTV-357T
- added D4, D5, D6: LED ON, LED_SMD:LED_0603_1608Metric, symbol Device:LED
- added R12, R13, R15: 180, PCM_Resistor_SMD_AKL:R_0603_1608Metric, symbol PCM_Resistor_US_AKL:R_0603
- added R14, R16, R18: 1k, PCM_Resistor_SMD_AKL:R_0603_1608Metric, symbol PCM_Resistor_US_AKL:R_0603
- added U11, U7, U8: LTV-357T, Package_SO:SO-4_4.4x3.6mm_P2.54mm, symbol Isolator:LTV-357T
Connections:
- net +3.3V: now also R12.1, R13.1, R15.1
- net GND: now also U11.2, U11.3, U7.2, U7.3, U8.2, U8.3
- new net: R18.2, U8.1
- new net: D5.2 (A), R13.2
- new net: D4.2 (A), R12.2
- new net: R16.2, U11.1
- new net: D6.2 (A), R15.2
- new net: R14.2, U7.1
- new net DIGITAL_IN_1: R16.1
- new net DIGITAL_IN_2: R14.1
- new net ESP32-S3_DIGITAL_IN_1: D4.1 (K), U11.4
- new net ESP32-S3_DIGITAL_IN_2: D5.1 (K), U7.4
- new net ESP32-S3_RUN_IN: D6.1 (K), U8.4
- new net RUN/STOP: R18.1
Other:
- note added: "Entrada DIGITAL #1"
- note added: "Entrada DIGITAL #2"
- note added: "RUN/STOP"
- note removed: "Entrada PNP #1"
- note removed: "Entrada PNP #2"

Commit message: Enrutando
Changed lines of the file:
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@@
-		)
-	)
-	(hierarchical_label "+3.3V"
-		(shape input)
-		(at 177.8 149.86 0)
-		(effects
-			(font
-				(size 1.27 1.27)
-			)
-			(justify left)
 		)
 	)
@@
 		)
 	)
-	(hierarchical_label "+3.3V"
-		(shape input)
-		(at 182.88 55.88 0)
-		(effects
-			(font
-				(size 1.27 1.27)
-			)
-			(justify left)
-		)
-	)
-	(hierarchical_label "+3.3V"
-		(shape input)
-		(at 181.61 100.33 0)
-		(effects
-			(font
-				(size 1.27 1.27)
-			)
-			(justify left)
-		)
-	)
 	(hierarchical_label "ESP32-S3_RUN_IN"
 		(shape output)
@@
 	)
 	(symbol
+		(lib_id "PCM_4ms_Power-symbol:+3.3V")
+		(at 181.61 100.33 270)
+		(unit 1)
+		(exclude_from_sim no)
+		(in_bom yes)
+		(on_board yes)
+		(dnp no)
+		(fields_autoplaced yes)
+		(property "Reference" "#PWR067"
+			(at 177.8 100.33 0)
+			(effects
+				(font
+					(size 1.27 1.27)
+				)
+				(hide yes)
+			)
+		)
+		(property "Value" "+3.3V"
+			(at 185.42 100.3299 90)
+			(effects
+				(font
+					(size 1.27 1.27)
+				)
+				(justify left)
+			)
+		)
+		(property "Footprint" ""
+			(at 181.61 100.33 0)
+			(effects
+				(font
+					(size 1.27 1.27)
+				)
+				(hide yes)
+			)
+		)
+		(property "Datasheet" ""
+			(at 181.61 100.33 0)
+			(effects
+				(font
+					(size 1.27 1.27)
+				)
+				(hide yes)
+			)
+		)
+		(property "Description" ""
+			(at 181.61 100.33 0)
+			(effects
+				(font
+					(size 1.27 1.27)
+				)
+				(hide yes)
+			)
+		)
+		(pin "1"
+		)
+		(instances
+			(project "zorionx_nivara"
+				(path "/c1255741-5652-463a-8cfd-bd2388ad7ef1/ee2c52cb-3406-40a8-8a05-a93f573fe34b/aa7002a9-6519-43d1-962e-402912e8a658"
+					(reference "#PWR067")
+					(unit 1)
+				)
+			)
+		)
+	)
+	(symbol
+		(lib_id "PCM_4ms_Power-symbol:+3.3V")
+		(at 177.8 149.86 270)
+		(unit 1)
+		(exclude_from_sim no)
+		(in_bom yes)
+		(on_board yes)
+		(dnp no)
+		(fields_autoplaced yes)
+		(property "Reference" "#PWR068"
+			(at 173.99 149.86 0)
+			(effects
+				(font
+					(size 1.27 1.27)
+				)
+				(hide yes)
+			)
+		)
+		(property "Value" "+3.3V"
+			(at 181.61 149.8599 90)
+			(effects
+				(font
+					(size 1.27 1.27)
+				)
+				(justify left)
+			)
+		)
+		(property "Footprint" ""
+			(at 177.8 149.86 0)
+			(effects
+				(font
+					(size 1.27 1.27)
+				)
+				(hide yes)
+			)
+		)
+		(property "Datasheet" ""
+			(at 177.8 149.86 0)
+			(effects
+				(font
+					(size 1.27 1.27)
+				)
+				(hide yes)
+			)
+		)
+		(property "Description" ""
+			(at 177.8 149.86 0)
+			(effects
+				(font
+					(size 1.27 1.27)
+				)
+				(hide yes)
+			)
+		)
+		(pin "1"
+		)
+		(instances
+			(project "zorionx_nivara"
+				(path "/c1255741-5652-463a-8cfd-bd2388ad7ef1/ee2c52cb-3406-40a8-8a05-a93f573fe34b/aa7002a9-6519-43d1-962e-402912e8a658"
+					(reference "#PWR068")
+					(unit 1)
+				)
+			)
+		)
+	)
+	(symbol
 		(lib_id "PCM_Resistor_US_AKL:R_0603")
 		(at 172.72 55.88 270)
@@
 					(unit 1)
 				)
+			)
+		)
+	)
+	(symbol
+		(lib_id "PCM_4ms_Power-symbol:+3.3V")
+		(at 182.88 55.88 270)
+		(unit 1)
+		(exclude_from_sim no)
+		(in_bom yes)
+		(on_board yes)
+		(dnp no)
+		(fields_autoplaced yes)
+		(property "Reference" "#PWR074"
+			(at 179.07 55.88 0)
+			(effects
+				(font
+					(size 1.27 1.27)
+				)
+				(hide yes)
+			)
+		)
+		(property "Value" "+3.3V"
+			(at 186.69 55.8799 90)
+			(effects
+				(font
+					(size 1.27 1.27)
+				)
+				(justify left)
+			)
+		)
+		(property "Footprint" ""
+			(at 182.88 55.88 0)
+			(effects
+				(font
+					(size 1.27 1.27)
+				)
+				(hide yes)
+			)
+		)
+		(property "Datasheet" ""
+			(at 182.88 55.88 0)
+			(effects
+				(font
+					(size 1.27 1.27)
+				)
+				(hide yes)
+			)
+		)
+		(property "Description" ""
+			(at 182.88 55.88 0)
+			(effects
+				(font
+					(size 1.27 1.27)
+				)
+				(hide yes)
+			)
+		)
+		(pin "1"
+		)
+		(instances
+			(project "zorionx_nivara"
+				(path "/c1255741-5652-463a-8cfd-bd2388ad7ef1/ee2c52cb-3406-40a8-8a05-a93f573fe34b/aa7002a9-6519-43d1-962e-402912e8a658"
+					(reference "#PWR074")
+					(unit 1)
+				)
