File: zorionx_nivara/Driver_RS485.kicad_sch (KiCad schematic)
At the start: 0 parts

Commit message: ultimo commit 1
Parts:
- added C7: 10uF, PCM_Capacitor_SMD_AKL:C_0603_1608Metric, symbol PCM_Capacitor_US_AKL:C_0603
- added D16: SMAJ5.0A, PCM_Diode_SMD_AKL:D_SMA, symbol PCM_Diode_TVS_AKL:SMAJ5.0A
- added D7: SMBJ12CA, PCM_Diode_SMD_AKL:D_SMB_TVS, symbol PCM_Diode_TVS_AKL:SMBJ12CA
- added D8: SM712, PCM_Package_TO_SOT_SMD_AKL:SOT-23, symbol PCM_Diode_TVS_AKL:SM712
- added R17, R19: R_0603, PCM_Resistor_SMD_AKL:R_0603_1608Metric, symbol PCM_Resistor_US_AKL:R_0603
- added U3: RSM3485ECHT_C2992406, EasyEDA:COMM-TH_8P-L19.5-W16.5-P2.54-BL, symbol EasyEDA:RSM3485ECHT_C2992406
Connections:
- net UART_IN: now also U3.3 (TXD)
- net UART_OUT: now also U3.4 (RXD)
- new net: D7.2 (A), D8.1 (A1), R17.1, U3.9 (A)
- new net: D7.1 (K), D8.2 (A2), R19.1, U3.8 (B)
- new net +3.3V: C7.1, D16.1 (K), U3.1 (VCC)
- new net GND: U3.5 (CON)
- new net GND1: C7.2, D16.2 (A), D8.3 (Com), U3.2 (GND)
- new net RS485_A: R17.2
- new net RS485_B: R19.2
Other:
- note added: "Transceptor RS-485 aislado"

Commit message: Salvado
Parts:
- removed U3: RSM3485ECHT_C2992406, EasyEDA:COMM-TH_8P-L19.5-W16.5-P2.54-BL, symbol EasyEDA:RSM3485ECHT_C2992406
- added U15: ~, Biblioteca_BryanFernandez_Huellas:YLPTEC RSM3485ECHT, symbol New_Library:RSM3485ECHT_C2992406
Connections:
- net +3.3V: now also U15.1 (VCC)
- net GND: now also U15.5 (CON)
- net GND1: now also U15.2 (GND)
- net UART_IN: now also U15.3 (TXD)
- net UART_OUT: now also U15.4 (RXD)
- net at D7.2 (A), D8.1 (A1), R17.1: now also U15.9 (A)
- net at D7.1 (K), D8.2 (A2), R19.1: now also U15.8 (B)
- no-connect marks 0 -> 1
Changed lines of the file:
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@@
 		(color 0 0 0 0)
 	)
-	(wire
-		(pts
-			(xy 137.16 96.52) (xy 134.62 96.52)
-		)
-		(stroke
-			(width 0)
-			(type default)
-		)
+	(no_connect
+		(at 132.08 88.9)
 	)
 	(wire
@@
 	(wire
 		(pts
-			(xy 134.62 91.44) (xy 146.05 91.44)
-		)
-		(stroke
-			(width 0)
-			(type default)
-		)
-	)
-	(wire
-		(pts
-			(xy 134.62 93.98) (xy 140.97 93.98)
-		)
-		(stroke
-			(width 0)
-			(type default)
-		)
-	)
-	(wire
-		(pts
 			(xy 96.52 104.14) (xy 96.52 101.6)
 		)
@@
 	(wire
 		(pts
+			(xy 132.08 93.98) (xy 140.97 93.98)
+		)
+		(stroke
+			(width 0)
+			(type default)
+		)
+	)
+	(wire
+		(pts
 			(xy 153.67 85.09) (xy 153.67 91.44)
 		)
@@
 	(wire
 		(pts
+			(xy 132.08 96.52) (xy 137.16 96.52)
+		)
+		(stroke
+			(width 0)
+			(type default)
+		)
+	)
+	(wire
+		(pts
 			(xy 110.49 93.98) (xy 110.49 106.68)
 		)
@@
 		(pts
 			(xy 143.51 115.57) (xy 143.51 118.11)
+		)
+		(stroke
+			(width 0)
+			(type default)
+		)
+	)
+	(wire
+		(pts
+			(xy 132.08 91.44) (xy 146.05 91.44)
 		)
 		(stroke
@@
 				(path "/c1255741-5652-463a-8cfd-bd2388ad7ef1/ee2c52cb-3406-40a8-8a05-a93f573fe34b/1f831b6c-7798-4c77-bf6f-f850ea2cc985"
 					(reference "C7")
+					(unit 1)
+				)
+			)
+		)
+	)
+	(symbol
+		(lib_id "New_Library:RSM3485ECHT_C2992406")
+		(at 113.03 86.36 0)
+		(unit 1)
+		(exclude_from_sim no)
+		(in_bom yes)
+		(on_board yes)
+		(dnp no)
+		(fields_autoplaced yes)
+		(property "Reference" "U15"
+			(at 123.19 82.55 0)
+			(effects
+				(font
+					(size 1.27 1.27)
+				)
+			)
+		)
+		(property "Value" "~"
+			(at 123.19 85.09 0)
+			(effects
+				(font
+					(size 1.27 1.27)
+				)
+			)
+		)
+		(property "Footprint" "Biblioteca_BryanFernandez_Huellas:YLPTEC RSM3485ECHT"
+			(at 113.03 86.36 0)
+			(effects
+				(font
+					(size 1.27 1.27)
+				)
+				(hide yes)
+			)
+		)
+		(property "Datasheet" ""
+			(at 113.03 86.36 0)
+			(effects
+				(font
+					(size 1.27 1.27)
+				)
+				(hide yes)
+			)
+		)
+		(property "Description" ""
+			(at 113.03 86.36 0)
+			(effects
+				(font
+					(size 1.27 1.27)
+				)
+				(hide yes)
+			)
+		)
+		(pin "8"
+		)
+		(pin "5"
+		)
+		(pin "3"
+		)
+		(pin "2"
+		)
+		(pin "10"
+		)
+		(pin "1"
+		)
+		(pin "4"
+		)
+		(pin "9"
+		)
+		(instances
+			(project ""
+				(path "/c1255741-5652-463a-8cfd-bd2388ad7ef1/ee2c52cb-3406-40a8-8a05-a93f573fe34b/1f831b6c-7798-4c77-bf6f-f850ea2cc985"
+					(reference "U15")
 					(unit 1)
 				)
@@
 		(dnp no)
 		(fields_autoplaced yes)
-		(property "Reference" "#PWR024"
+		(property "Reference" "#PWR0101"
 			(at 96.52 110.49 0)
 			(effects
@@
 			(project "zorionx_nivara"
 				(path "/c1255741-5652-463a-8cfd-bd2388ad7ef1/ee2c52cb-3406-40a8-8a05-a93f573fe34b/1f831b6c-7798-4c77-bf6f-f850ea2cc985"
-					(reference "#PWR024")
+					(reference "#PWR0101")
 					(unit 1)
 				)
@@
 					(unit 1)
 				)
-			)
-		)
-	)
-	(symbol
-		(lib_id "EasyEDA:RSM3485ECHT_C2992406")
-		(at 124.46 92.71 0)
-		(unit 1)
-		(exclude_from_sim no)
-		(in_bom yes)
-		(on_board yes)
-		(dnp no)
-		(fields_autoplaced yes)
-		(property "Reference" "U3"
-			(at 124.46 81.28 0)
-			(effects
-				(font
-					(size 1.27 1.27)
-				)
-			)
-		)
-		(property "Value" "RSM3485ECHT_C2992406"
-			(at 124.46 83.82 0)
-			(effects
-				(font
-					(size 1.27 1.27)
-				)
-			)
-		)
-		(property "Footprint" "EasyEDA:COMM-TH_8P-L19.5-W16.5-P2.54-BL"
-			(at 124.46 104.14 0)
-			(effects
-				(font
-					(size 1.27 1.27)
-				)
-				(hide yes)
-			)
-		)
-		(property "Datasheet" "https://lcsc.com/product-detail/RS485-Bus-Modules_VISOM-RSM3485ECHT_C882099.html?s_z=n_RSM3485ECHT_C2992406"
-			(at 124.46 92.71 0)
-			(effects
-				(font
-					(size 1.27 1.27)
-				)
-				(hide yes)
-			)
-		)
-		(property "Description" "500Kbps 256 No DIP-8 RS485 Bus Modules ROHS"
-			(at 124.46 92.71 0)
-			(effects
-				(font
-					(size 1.27 1.27)
-				)
-				(hide yes)
-			)
-		)
-		(property "Part Number #" "C882099"
-			(at 124.46 106.68 0)
-			(effects
-				(font
-					(size 1.27 1.27)
-				)
-				(hide yes)
-			)
-		)
-		(pin "4"
-		)
-		(pin "9"
-		)
-		(pin "1"
-		)
-		(pin "3"
-		)
-		(pin "10"
-		)
-		(pin "2"
-		)
-		(pin "8"
-		)
-		(pin "5"
-		)
-		(instances
-			(project "zorionx_nivara"
-				(path "/c1255741-5652-463a-8cfd-bd2388ad7ef1/ee2c52cb-3406-40a8-8a05-a93f573fe34b/1f831b6c-7798-4c77-bf6f-f850ea2cc985"
-					(reference "U3")
-					(unit 1)
-				)

Commit message: Salvado1
Parts:
- U15: value ~ -> RSM3485ECHT_C2992406
Changed lines of the file:
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@@
 			)
 		)
-		(property "Value" "~"
+		(property "Value" "RSM3485ECHT_C2992406"
 			(at 123.19 85.09 0)
 			(effects

Commit message: Enrutando
Changed lines of the file:
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@@
-		)
-	)
-	(hierarchical_label "+3.3V"
-		(shape input)
-		(at 85.09 88.9 180)
-		(effects
-			(font
-				(size 1.27 1.27)
-			)
-			(justify right)
 		)
 	)
@@
 					(unit 1)
 				)
+			)
+		)
+	)
+	(symbol
+		(lib_id "PCM_4ms_Power-symbol:+3.3V")
+		(at 85.09 88.9 90)
+		(unit 1)
+		(exclude_from_sim no)
+		(in_bom yes)
+		(on_board yes)
+		(dnp no)
+		(fields_autoplaced yes)
+		(property "Reference" "#PWR072"
+			(at 88.9 88.9 0)
+			(effects
+				(font
+					(size 1.27 1.27)
+				)
+				(hide yes)
+			)
+		)
+		(property "Value" "+3.3V"
+			(at 81.28 88.8999 90)
+			(effects
+				(font
+					(size 1.27 1.27)
+				)
+				(justify left)
+			)
+		)
+		(property "Footprint" ""
+			(at 85.09 88.9 0)
+			(effects
+				(font
+					(size 1.27 1.27)
+				)
+				(hide yes)
+			)
+		)
+		(property "Datasheet" ""
+			(at 85.09 88.9 0)
+			(effects
+				(font
+					(size 1.27 1.27)
+				)
+				(hide yes)
+			)
+		)
+		(property "Description" ""
+			(at 85.09 88.9 0)
+			(effects
+				(font
+					(size 1.27 1.27)
+				)
+				(hide yes)
+			)
+		)
+		(pin "1"
+		)
+		(instances
+			(project "zorionx_nivara"
+				(path "/c1255741-5652-463a-8cfd-bd2388ad7ef1/ee2c52cb-3406-40a8-8a05-a93f573fe34b/1f831b6c-7798-4c77-bf6f-f850ea2cc985"
+					(reference "#PWR072")
+					(unit 1)
+				)

Commit message: Enrutando_finalizando1
Parts:
- R17, R19: value R_0603 -> 47K
Connections:
- net GND1 is gone; now on net GND: C7.2, D16.2 (A), D8.3 (Com), U15.2 (GND)
Changed lines of the file:
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@@
+	(symbol
+		(lib_id "power:GND")
+		(at 143.51 118.11 0)
+		(unit 1)
+		(exclude_from_sim no)
+		(in_bom yes)
+		(on_board yes)
+		(dnp no)
+		(fields_autoplaced yes)
+		(property "Reference" "#PWR024"
+			(at 143.51 124.46 0)
+			(effects
+				(font
+					(size 1.27 1.27)
+				)
+				(hide yes)
+			)
+		)
+		(property "Value" "GND"
+			(at 143.51 123.19 0)
+			(effects
+				(font
+					(size 1.27 1.27)
+				)
+			)
+		)
+		(property "Footprint" ""
+			(at 143.51 118.11 0)
+			(effects
+				(font
+					(size 1.27 1.27)
+				)
+				(hide yes)
+			)
+		)
+		(property "Datasheet" ""
+			(at 143.51 118.11 0)
+			(effects
+				(font
+					(size 1.27 1.27)
+				)
+				(hide yes)
+			)
+		)
+		(property "Description" "Power symbol creates a global label with name \"GND\" , ground"
+			(at 143.51 118.11 0)
+			(effects
+				(font
+					(size 1.27 1.27)
+				)
+				(hide yes)
+			)
+		)
+		(pin "1"
+		)
+		(instances
+			(project "zorionx_nivara"
+				(path "/c1255741-5652-463a-8cfd-bd2388ad7ef1/ee2c52cb-3406-40a8-8a05-a93f573fe34b/1f831b6c-7798-4c77-bf6f-f850ea2cc985"
+					(reference "#PWR024")
+					(unit 1)
+				)
+			)
+		)
+	)
 	(symbol
 		(lib_id "power:GND")
@@
 	)
 	(symbol
-		(lib_id "power:GND")
-		(at 143.51 118.11 0)
-		(unit 1)
-		(exclude_from_sim no)
-		(in_bom yes)
-		(on_board yes)
-		(dnp no)
-		(fields_autoplaced yes)
-		(property "Reference" "#PWR024"
-			(at 143.51 124.46 0)
-			(effects
-				(font
-					(size 1.27 1.27)
-				)
-				(hide yes)
-			)
-		)
-		(property "Value" "GND1"
-			(at 143.51 123.19 0)
-			(effects
-				(font
-					(size 1.27 1.27)
-				)
-			)
-		)
-		(property "Footprint" ""
-			(at 143.51 118.11 0)
-			(effects
-				(font
-					(size 1.27 1.27)
-				)
-				(hide yes)
-			)
-		)
-		(property "Datasheet" ""
-			(at 143.51 118.11 0)
-			(effects
-				(font
-					(size 1.27 1.27)
-				)
-				(hide yes)
-			)
-		)
-		(property "Description" "Power symbol creates a global label with name \"GND\" , ground"
-			(at 143.51 118.11 0)
-			(effects
-				(font
-					(size 1.27 1.27)
-				)
-				(hide yes)
-			)
-		)
-		(pin "1"
-		)
-		(instances
-			(project "zorionx_nivara"
-				(path "/c1255741-5652-463a-8cfd-bd2388ad7ef1/ee2c52cb-3406-40a8-8a05-a93f573fe34b/1f831b6c-7798-4c77-bf6f-f850ea2cc985"
-					(reference "#PWR024")
-					(unit 1)
-				)
-			)
-		)
-	)
-	(symbol
 		(lib_id "PCM_Resistor_US_AKL:R_0603")
 		(at 158.75 91.44 90)
@@
 			)
 		)
-		(property "Value" "R_0603"
+		(property "Value" "47K"
 			(at 158.75 87.63 90)
 			(effects
@@
 		(dnp no)
 		(fields_autoplaced yes)
-		(property "Reference" "#PWR0101"
+		(property "Reference" "#PWR046"
 			(at 96.52 110.49 0)
 			(effects
@@
 			)
 		)
-		(property "Value" "GND1"
+		(property "Value" "GND"
 			(at 96.52 109.22 0)
 			(effects
@@
 		)
 		(instances
-			(project "zorionx_nivara"
-				(path "/c1255741-5652-463a-8cfd-bd2388ad7ef1/ee2c52cb-3406-40a8-8a05-a93f573fe34b/1f831b6c-7798-4c77-bf6f-f850ea2cc985"
-					(reference "#PWR0101")
+			(project ""
+				(path "/c1255741-5652-463a-8cfd-bd2388ad7ef1/ee2c52cb-3406-40a8-8a05-a93f573fe34b/1f831b6c-7798-4c77-bf6f-f850ea2cc985"
+					(reference "#PWR046")
 					(unit 1)
 				)
@@
 			)
 		)
-		(property "Value" "R_0603"
+		(property "Value" "47K"
 			(at 167.64 90.17 90)
 			(effects
