File: zorionx_nivara/Output_NPN.kicad_sch (KiCad schematic)
At the start: 0 parts

Commit message: ultimo commit 1
Parts:
- added D27, D9: LED ON, LED_SMD:LED_0603_1608Metric, symbol Device:LED
- added Q1, Q2: AO3407A, PCM_Package_TO_SOT_SMD_AKL:SOT-23, symbol PCM_Transistor_MOSFET_AKL:AO3407A
- added R20, R21, R23, R25: 100, PCM_Resistor_SMD_AKL:R_0603_1608Metric, symbol PCM_Resistor_US_AKL:R_0603
- added R22, R24: 100k, PCM_Resistor_SMD_AKL:R_0603_1608Metric, symbol PCM_Resistor_US_AKL:R_0603
- added R26, R54: 1.5k, PCM_Resistor_SMD_AKL:R_0603_1608Metric, symbol PCM_Resistor_US_AKL:R_0603
- added U10, U9: LTV-357T, Package_SO:SO-4_4.4x3.6mm_P2.54mm, symbol Isolator:LTV-357T
Connections:
- new net: R23.2, U10.1
- new net: R25.2, U10.4
- new net: Q2.1 (G), R24.2, R25.1
- new net: R20.2, U9.1
- new net: R21.2, U9.4
- new net: D27.2 (A), R54.2
- new net: Q1.1 (G), R21.1, R22.2
- new net: D9.2 (A), R26.2
- new net ESP32-S3_NPN_OUT_1: R20.1
- new net ESP32-S3_NPN_OUT_2: R23.1
- new net GND1: U10.2, U9.2
- new net GND2: D27.1 (K), D9.1 (K), U10.3, U9.3
- new net NPN_OUT_1: Q1.3 (D), R54.1
- new net NPN_OUT_2: Q2.3 (D), R26.1
- new net VCC2: Q1.2 (S), Q2.2 (S), R22.1, R24.1
Other:
- note added: "Salida NPN #1"
- note added: "Salida NPN #2"

Commit message: Enrutando_finalizando1
Connections:
- net GND2 is gone; now on net GND: D27.1 (K), D9.1 (K), U10.3, U9.3
- net GND1 renamed GND
- net VCC2 renamed VCC
