File: zorionx_nivara/Output_PNP.kicad_sch (KiCad schematic)
At the start: 14 parts, among them Q3 IRLML0040, Q4 IRLML0040, U12 LTV-357T, U14 LTV-357T

Commit message: Enrutando_finalizando1
Connections:
- net GND2 is gone; now on net GND: Q3.2 (S), Q4.2 (S), R29.1, R32.1, U12.3, U14.3
- net GND1 renamed GND
- net VCC2 renamed VCC
