File: zorionx_nivara/zorionx_nivara.kicad_sch (KiCad schematic)
At the start: 13 parts, among them J1 Screw_Terminal_3_P5.00mm, J12 Screw_Terminal_4_P5.00mm, J13 Screw_Terminal_6_P5.00mm, J14 Screw_Terminal_2_P5.00mm, J2 Screw_Terminal_2_P5.00mm, J3 Screw_Terminal_2_P5.00mm, J4 Screw_Terminal_4_P5.00mm, J5 Screw_Terminal_2_P5.00mm, J6 Screw_Terminal_2_P5.00mm, J9 Screw_Terminal_3_P5.00mm

Commit message: ultimo commit 1
Connections:
- net GND: now also H1.1, H2.1
Other:
- title: ZorionX - Nivara -> ZorionX - Nivara / Bryan S. Fernandez M. 2022-0917
- moved on the sheet: AE1, H1, H2, J1, J12, J13, J14, J2, J3, J4, J5, J6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

Commit message: Enrutando
Parts:
- J1: value Screw_Terminal_3_P5.00mm -> Salidas Analogicas
- J12: value Screw_Terminal_4_P5.00mm -> Salidas NPN/PNP
- J13: value Screw_Terminal_6_P5.00mm -> Reles
- J14: value Screw_Terminal_2_P5.00mm -> Entrada NPN
- J2: value Screw_Terminal_2_P5.00mm -> Entrada PNP
- J3: value Screw_Terminal_2_P5.00mm -> Alimentacion
- J4: value Screw_Terminal_4_P5.00mm -> Entradas Analogicas
- J5: value Screw_Terminal_2_P5.00mm -> Entradas digitales
- J6: value Screw_Terminal_2_P5.00mm -> RUN/STOP
- J9: value Screw_Terminal_3_P5.00mm -> RS-485
Connections:
- net board_zorionx-nivara/D_IN1 renamed board_zorionx-nivara/DIGITAL_IN1
- net board_zorionx-nivara/D_IN2 renamed board_zorionx-nivara/DIGITAL_IN2
Other:
- sheet board_zorionx-nivara ports: added DIGITAL_IN1, DIGITAL_IN2; removed D_IN1, D_IN2
Changed lines of the file:
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@@
 			)
 		)
-		(property "Value" "Screw_Terminal_2_P5.00mm"
+		(property "Value" "Entrada NPN"
 			(at 98.425 121.92 0)
 			(effects
@@
 			)
 		)
-		(property "Value" "Screw_Terminal_4_P5.00mm"
+		(property "Value" "Salidas NPN/PNP"
 			(at 151.13 160.0199 0)
 			(effects
@@
 			)
 		)
-		(property "Value" "Screw_Terminal_4_P5.00mm"
+		(property "Value" "Entradas Analogicas"
 			(at 98.425 157.48 0)
 			(effects
@@
 			)
 		)
-		(property "Value" "Screw_Terminal_2_P5.00mm"
+		(property "Value" "RUN/STOP"
 			(at 98.425 186.69 0)
 			(effects
@@
 			)
 		)
-		(property "Value" "Screw_Terminal_3_P5.00mm"
+		(property "Value" "RS-485"
 			(at 151.13 128.2699 0)
 			(effects
@@
 			)
 		)
-		(property "Value" "Screw_Terminal_3_P5.00mm"
+		(property "Value" "Salidas Analogicas"
 			(at 151.13 142.2399 0)
 			(effects
@@
 			)
 		)
-		(property "Value" "Screw_Terminal_2_P5.00mm"
+		(property "Value" "Alimentacion"
 			(at 117.475 113.03 0)
 			(effects
@@
 			)
 		)
-		(property "Value" "Screw_Terminal_2_P5.00mm"
+		(property "Value" "Entrada PNP"
 			(at 98.425 130.81 0)
 			(effects
@@
 			)
 		)
-		(property "Value" "Screw_Terminal_6_P5.00mm"
+		(property "Value" "Reles"
 			(at 151.13 177.7999 0)
 			(effects
@@
 			)
 		)
-		(property "Value" "Screw_Terminal_2_P5.00mm"
+		(property "Value" "Entradas digitales"
 			(at 98.425 161.29 0)
 			(effects
@@
 			)
 		)
-		(pin "D_IN1" input
-			(at 106.68 165.1 180)
-			(effects
-				(font
-					(size 1.27 1.27)
-				)
-				(justify left)
-			)
-		)
-		(pin "D_IN2" input
-			(at 106.68 167.64 180)
-			(effects
-				(font
-					(size 1.27 1.27)
-				)
-				(justify left)
-			)
-		)
 		(pin "NPN_IN_1" input
 			(at 106.68 125.73 180)
@@
 			)
 		)
+		(pin "DIGITAL_IN1" input
+			(at 106.68 165.1 180)
+			(effects
+				(font
+					(size 1.27 1.27)
+				)
+				(justify left)
+			)
+		)
+		(pin "DIGITAL_IN2" input
+			(at 106.68 167.64 180)
+			(effects
+				(font
+					(size 1.27 1.27)
+				)
+				(justify left)
+			)
+		)

Commit message: Enrutando_finalizando1
Connections:
- net board_zorionx-nivara/RLY1_NC: now also J13.3; no longer J13.1
- net board_zorionx-nivara/RLY1_NO: now also J13.1; no longer J13.3
- net board_zorionx-nivara/RLY2_C: now also J13.4; no longer J13.5
- net board_zorionx-nivara/RLY2_NC: now also J13.6; no longer J13.4
- net board_zorionx-nivara/RLY2_NO: now also J13.5; no longer J13.6
