File: zorionx_nivara/board_zorionx-nivara.kicad_sch (KiCad schematic)
At the start: 3 parts, among them U1 ESP32-S3-WROOM-1

Commit message: ultimo commit 1
Parts:
- R2: value 22K -> ~
Connections:
- net Driver_RS485/UART_IN: now also U1.10 (IO17); no longer U1.37 (TXD0)
- net Driver_RS485/UART_OUT: now also U1.11 (IO18); no longer U1.36 (RXD0)
Other:
- sheet Input_NPN renamed INPUTS_NPN
- sheet Input_PNP renamed INPUTS_PNP
- sheet PowerSupply renamed PowerSupply +3V
- added sheet ANALOG_IN (ANALOG_IN.kicad_sch)
- added sheet DIGITAL_IN (DIGITAL_IN.kicad_sch)
- sheet INPUTS_NPN ports: added +3.3V, ESP32-S3_NPN_IN_1, ESP32-S3_NPN_IN_2, NPN_IN_1, NPN_IN_2, VCC; removed none
- sheet INPUTS_PNP ports: added +3.3V, ESP32-S3_PNP_IN_1, ESP32-S3_PNP_IN_2, PNP_IN_1, PNP_IN_2; removed none
- sheet Output_NPN ports: added ESP32-S3_NPN_OUT_1, ESP32-S3_NPN_OUT_2, NPN_OUT_1, NPN_OUT_2, VCC2; removed none
- sheet Output_PNP ports: added ESP32-S3_PNP_OUT_1, ESP32-S3_PNP_OUT_2, PNP_OUT_1, PNP_OUT_2, VCC2; removed none
- sheet PowerSupply +3V ports: added +3.3V, VCC; removed none
- moved on the sheet: C5, R2, U1

Commit message: Salvado
Connections:
- net ANALOG_IN/ESP32-S3_4-20_IN: now also U1.15 (IO3)
- net ANALOG_IN/ESP32-S3_A0_10_IN_1: now also U1.39 (IO1)
- net ANALOG_IN/ESP32-S3_A0_32_IN_1: now also U1.38 (IO2)
- net DIGITAL_IN/ESP32-S3_DIGITAL_IN_1: now also U1.12 (IO8)
- net DIGITAL_IN/ESP32-S3_DIGITAL_IN_2: now also U1.17 (IO9)
- net DIGITAL_IN/ESP32-S3_RUN_IN: now also U1.18 (IO10)
- net INPUTS_NPN/ESP32-S3_NPN_IN_1: now also U1.27 (IO0)
- net INPUTS_NPN/ESP32-S3_NPN_IN_2: now also U1.4 (IO4)
- net INPUTS_PNP/ESP32-S3_PNP_IN_1: now also U1.5 (IO5)
- net INPUTS_PNP/ESP32-S3_PNP_IN_2: now also U1.6 (IO6)
- net Output_NPN/ESP32-S3_NPN_OUT_1: now also U1.32 (IO39)
- net Output_NPN/ESP32-S3_NPN_OUT_2: now also U1.33 (IO40)
- net Output_PNP/ESP32-S3_PNP_OUT_1: now also U1.22 (IO14)
- net Output_PNP/ESP32-S3_PNP_OUT_2: now also U1.21 (IO13)
- net RELAY_#1_#2/ESP32-S3_RY1: now reaches U1.19 (IO11)
- net RELAY_#1_#2/ESP32-S3_RLY2: now reaches U1.20 (IO12)
- net ANALOG_OUT/ESP32-S3_SEL_VOUT: now reaches U1.7 (IO7)
- net ANALOG_OUT/SDA_V: now reaches U1.8 (IO15)
- net ANALOG_OUT/SCLK_V: now reaches U1.9 (IO16)
Other:
- added sheet ANALOG_OUT (ANALOG_OUT.kicad_sch)
- added sheet RELAY_#1_#2 (RELAY_#1_#2.kicad_sch)
- moved on the sheet: C5, R2, U1

Commit message: Enrutando
Other:
- sheet ANALOG_IN ports: added none; removed +3.3V
- sheet ANALOG_OUT ports: added none; removed +3.3V
- sheet DIGITAL_IN ports: added none; removed +3.3V
- sheet INPUTS_NPN ports: added none; removed +3.3V
- sheet INPUTS_PNP ports: added none; removed +3.3V
- sheet PowerSupply +3V ports: added none; removed +3.3V

Commit message: Enrutando_finalizando1
Connections:
- net ANALOG_OUT/SCLK_C: now also U1.25 (IO48)
- net ANALOG_OUT/SDA_C: now also U1.24 (IO47)
Other:
- sheet INPUTS_NPN ports: added none; removed VCC
- sheet Output_PNP ports: added none; removed VCC2
- sheet PowerSupply +3V ports: added none; removed VCC
- sheet RELAY_#1_#2 ports: added none; removed VCC1

Commit message: Enrutando_finalizado2
Parts:
- added C16: 1uF, PCM_Capacitor_SMD_AKL:C_0603_1608Metric, symbol PCM_Capacitor_AKL:C_0603
Connections:
- net +3.3V: now also C16.1
- net GND: now also C16.2
Other:
- sheet Driver_RS485 ports: added RS485_A, RS485_B; removed RS485-A, RS485-B
Changed lines of the file:
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@@
+	(wire
+		(pts
+			(xy 168.91 45.72) (xy 168.91 50.8)
+		)
+		(stroke
+			(width 0)
+			(type default)
+		)
+	)
 	(wire
 		(pts
@@
 	(wire
 		(pts
+			(xy 168.91 34.29) (xy 179.07 34.29)
+		)
+		(stroke
+			(width 0)
+			(type default)
+		)
+	)
+	(wire
+		(pts
 			(xy 171.45 156.21) (xy 193.04 156.21)
 		)
@@
 	(wire
 		(pts
+			(xy 168.91 50.8) (xy 160.02 50.8)
+		)
+		(stroke
+			(width 0)
+			(type default)
+		)
+	)
+	(wire
+		(pts
 			(xy 41.91 44.45) (xy 41.91 46.99)
 		)
@@
 	(wire
 		(pts
+			(xy 179.07 34.29) (xy 179.07 38.1)
+		)
+		(stroke
+			(width 0)
+			(type default)
+		)
+	)
+	(wire
+		(pts
 			(xy 133.35 91.44) (xy 144.78 91.44)
 		)
@@
 		(pts
 			(xy 193.04 156.21) (xy 193.04 114.3)
+		)
+		(stroke
+			(width 0)
+			(type default)
+		)
+	)
+	(wire
+		(pts
+			(xy 168.91 38.1) (xy 168.91 34.29)
 		)
 		(stroke
@@
 			)
 			(justify left)
+		)
+	)
+	(symbol
+		(lib_id "PCM_Capacitor_AKL:C_0603")
+		(at 168.91 41.91 0)
+		(mirror x)
+		(unit 1)
+		(exclude_from_sim no)
+		(in_bom yes)
+		(on_board yes)
+		(dnp no)
+		(property "Reference" "C16"
+			(at 176.276 40.386 90)
+			(effects
+				(font
+					(size 1.27 1.27)
+				)
+				(justify left)
+			)
+		)
+		(property "Value" "1uF"
+			(at 173.736 40.386 90)
+			(effects
+				(font
+					(size 1.27 1.27)
+				)
+				(justify left)
+			)
+		)
+		(property "Footprint" "PCM_Capacitor_SMD_AKL:C_0603_1608Metric"
+			(at 169.8752 38.1 0)
+			(effects
+				(font
+					(size 1.27 1.27)
+				)
+				(hide yes)
+			)
+		)
+		(property "Datasheet" "~"
+			(at 168.91 41.91 0)
+			(effects
+				(font
+					(size 1.27 1.27)
+				)
+				(hide yes)
+			)
+		)
+		(property "Description" "SMD 0603 MLCC capacitor, Alternate KiCad Library"
+			(at 168.91 41.91 0)
+			(effects
+				(font
+					(size 1.27 1.27)
+				)
+				(hide yes)
+			)
+		)
+		(pin "1"
+		)
+		(pin "2"
+		)
+		(instances
+			(project "zorionx_nivara"
+				(path "/c1255741-5652-463a-8cfd-bd2388ad7ef1/ee2c52cb-3406-40a8-8a05-a93f573fe34b"
+					(reference "C16")
+					(unit 1)
+				)
+			)
 		)
 	)
@@
 	)
 	(symbol
+		(lib_id "power:GND")
+		(at 179.07 38.1 0)
+		(unit 1)
+		(exclude_from_sim no)
+		(in_bom yes)
+		(on_board yes)
+		(dnp no)
+		(property "Reference" "#PWR088"
+			(at 179.07 44.45 0)
+			(effects
+				(font
+					(size 1.27 1.27)
+				)
+				(hide yes)
+			)
+		)
+		(property "Value" "GND"
+			(at 178.816 43.434 0)
+			(effects
+				(font
+					(size 1.27 1.27)
+				)
+			)
+		)
+		(property "Footprint" ""
+			(at 179.07 38.1 0)
+			(effects
+				(font
+					(size 1.27 1.27)
+				)
+				(hide yes)
+			)
+		)
+		(property "Datasheet" ""
+			(at 179.07 38.1 0)
+			(effects
+				(font
+					(size 1.27 1.27)
+				)
+				(hide yes)
+			)
+		)
+		(property "Description" "Power symbol creates a global label with name \"GND\" , ground"
+			(at 179.07 38.1 0)
+			(effects
+				(font
+					(size 1.27 1.27)
+				)
+				(hide yes)
+			)
+		)
+		(pin "1"
+		)
+		(instances
+			(project "zorionx_nivara"
+				(path "/c1255741-5652-463a-8cfd-bd2388ad7ef1/ee2c52cb-3406-40a8-8a05-a93f573fe34b"
+					(reference "#PWR088")
+					(unit 1)
+				)
+			)
+		)
+	)
+	(symbol
 		(lib_id "PCM_Capacitor_AKL:C_0603")
 		(at 142.24 41.91 0)
@@
 			)
 		)
-		(pin "RS485-A" output
-			(at 218.44 50.8 0)
-			(effects
-				(font
-					(size 1.27 1.27)
-				)
-				(justify right)
-			)
-		)
-		(pin "RS485-B" output
-			(at 218.44 53.34 0)
-			(effects
-				(font
-					(size 1.27 1.27)
-				)
-				(justify right)
-			)
-		)
 		(pin "UART_IN" input
 			(at 189.23 50.8 180)
@@
 			)
 		)
+		(pin "RS485_A" bidirectional
+			(at 218.44 50.8 0)
+			(effects
+				(font
+					(size 1.27 1.27)
+				)
+				(justify right)
+			)
+		)
+		(pin "RS485_B" bidirectional
+			(at 218.44 53.34 0)
+			(effects
+				(font
+					(size 1.27 1.27)
+				)
+				(justify right)
+			)
+		)
